Commit message: fixed caster_front

File: src/wheeled-robot-description/urdf/wheeled-robot.xacro (robot description, xacro)
@@ -69,5 +69,5 @@
     <collision name="collision_chassis">
       <geometry>
-        <box size="0.5 0.3 0.01"/>
+        <box size="0.5 0.3 0.05"/>
       </geometry>
     </collision>
@@ -75,10 +75,10 @@
       <origin rpy="0 0 0" xyz="0 0 0"/>
       <geometry>
-        <box size="0.5 0.3 0.01"/>
+        <box size="0.5 0.3 0.05"/>
       </geometry>
       <material name="blue"/>
     </visual>
     <!-- caster front -->
-    <collision name="caster_front_collision">
+    <!-- <collision name="caster_front_collision">
       <origin rpy=" 0 0 0" xyz="0.2 0 -0.04"/>
       <geometry>
@@ -101,14 +101,49 @@
         <sphere radius="0.04"/>
       </geometry>
+    </visual> -->
+    </link>
+  <link name = "caster_front">
+    <inertial>
+      <mass value="0.1"/>
+      <!-- <origin rpy="0 0 0" xyz="0 0 0"/> -->
+      <inertia ixx="3.569e-7" ixy="0.000e+0" ixz="0.000e+0" iyy="5.344e-7" iyz="0.000e+0" izz="3.569e-7"/>
+    </inertial>
+    <collision name="caster_front_collision">
+      <!-- <origin rpy=" 0 0 0" xyz="0.2 0 -0.04"/> -->
+      <geometry>
+        <sphere radius="0.04"/>
+      </geometry>
+      <surface>
+        <friction>
+          <ode>
+            <mu>0</mu>
+            <mu2>0</mu2>
+            <slip1>1.0</slip1>
+            <slip2>1.0</slip2>
+          </ode>
+        </friction>
+      </surface>
+    </collision>
+    <visual name="caster_front_visual">
+      <!-- <origin rpy=" 0 0 0" xyz="0.2 0 -0.04"/> -->
+      <geometry>
+        <sphere radius="0.04"/>
+      </geometry>
     </visual>
-    </link>
+  </link>
+  <joint name = "caster_front_to_chassis" type = "continuous">
+    <parent link="link_chassis"/>
+    <child link="caster_front"/>
+    <origin rpy=" 0 0 0" xyz="0.2 0 -0.04"/>
+    <axis xyz="1 1 0"/>
+  </joint>
   <!-- Create wheel right -->
   <xacro:link_wheel name="link_right_wheel" />
   <!--   Joint for right wheel  -->
-  <xacro:joint_wheel name="joint_right_wheel"  child="link_right_wheel"  origin_xyz="-0.05 0.17 0"  />
+  <xacro:joint_wheel name="joint_right_wheel"  child="link_right_wheel"  origin_xyz="-0.13 -0.17 0"  />
   <!-- Left Wheel link -->
   <xacro:link_wheel name="link_left_wheel" />
-  <!--   Joint for right wheel  -->
-  <xacro:joint_wheel name="joint_left_wheel"   child="link_left_wheel"   origin_xyz="-0.05 -0.17 0"  />
+  <!--   Joint for left wheel  -->
+  <xacro:joint_wheel name="joint_left_wheel"   child="link_left_wheel"   origin_xyz="-0.13 0.17 0"  />
   <link name="sensor_laser">
     <inertial>
