Commit message: added camera/aruco_world

File: src/wheeled-robot-description/urdf/macro.xacro (robot description, xacro)
@@ -32,3 +32,21 @@
       </joint>
     </xacro:macro>
+    <macro name="cylinder_inertia" params="m r h">
+      <inertia  ixx="${m*(3*r*r+h*h)/12}" ixy = "0" ixz = "0"
+        iyy="${m*(3*r*r+h*h)/12}" iyz = "0"
+        izz="${m*r*r/2}"
+      />
+    </macro>
+    <macro name="box_inertia" params="m x y z">
+      <inertia  ixx="${m*(y*y+z*z)/12}" ixy = "0" ixz = "0"
+        iyy="${m*(x*x+z*z)/12}" iyz = "0"
+        izz="${m*(x*x+z*z)/12}"
+      />
+    </macro>
+    <macro name="sphere_inertia" params="m r">
+      <inertia  ixx="${2*m*r*r/5}" ixy = "0" ixz = "0"
+        iyy="${2*m*r*r/5}" iyz = "0"
+        izz="${2*m*r*r/5}"
+      />
+    </macro>
 </robot>

File: src/wheeled-robot-description/urdf/wheeled-robot.xacro (robot description, xacro)
@@ -1,62 +1,9 @@
 <?xml version="1.0" ?>
 <robot name="wheeled-robot" xmlns:xacro="https://www.ros.org/wiki/xacro" >
+<xacro:property name = "cameraSize" value = "0.05" />
+<xacro:property name = "cameraMass" value = "0.1" />
 <xacro:include filename="$(find wheeled-robot-description)/urdf/materials.xacro" />
-<!-- <xacro:include filename="$(find wheeled-robot-description)/urdf/robot.gazebo" /> -->
+<xacro:include filename="$(find wheeled-robot-description)/urdf/robot.gazebo" />
 <xacro:include filename="$(find wheeled-robot-description)/urdf/macro.xacro" />
-  <gazebo reference="link_chassis">
-    <material>Gazebo/Orange</material>
-  </gazebo>
-  <gazebo reference="link_left_wheel">
-    <material>Gazebo/Blue</material>
-  </gazebo>
-  <gazebo reference="link_right_wheel">
-    <material>Gazebo/Blue</material>
-  </gazebo>
-    <gazebo>
-    <plugin filename="libgazebo_ros_diff_drive.so" name="differential_drive_controller">
-      <alwaysOn>true</alwaysOn>
-      <updateRate>20</updateRate>
-      <leftJoint>joint_left_wheel</leftJoint>
-      <rightJoint>joint_right_wheel</rightJoint>
-      <wheelSeparation>0.34</wheelSeparation>
-      <wheelDiameter>0.2</wheelDiameter>
-      <torque>0.1</torque>
-      <commandTopic>cmd_vel</commandTopic>
-      <odometryTopic>odom</odometryTopic>
-      <odometryFrame>odom</odometryFrame>
-      <robotBaseFrame>link_chassis</robotBaseFrame>
-    </plugin>
-  </gazebo>
-  <gazebo reference="sensor_laser">
-    <sensor type="ray" name="head_hokuyo_sensor">
-      <pose>0 0 0 0 0 0</pose>
-      <visualize>false</visualize>
-      <update_rate>20</update_rate>
-      <ray>
-        <scan>
-          <horizontal>
-            <samples>720</samples>
-            <resolution>1</resolution>
-            <min_angle>-1.570796</min_angle>
-            <max_angle>1.570796</max_angle>
-          </horizontal>
-        </scan>
-        <range>
-          <min>0.10</min>
-          <max>10.0</max>
-          <resolution>0.01</resolution>
-        </range>
-        <noise>
-          <type>gaussian</type>
-          <mean>0.0</mean>
-          <stddev>0.01</stddev>
-        </noise>
-      </ray>
-      <plugin name="gazebo_ros_head_hokuyo_controller" filename="libgazebo_ros_laser.so">
-        <topicName>/m2wr/laser/scan</topicName>
-        <frameName>sensor_laser</frameName>
-      </plugin>
-    </sensor>
-  </gazebo>
   <link name="link_chassis">
     <!-- pose and inertial -->
@@ -79,27 +26,4 @@
       <material name="blue"/>
     </visual>
-    <!-- caster front -->
-    <!-- <collision name="caster_front_collision">
-      <origin rpy=" 0 0 0" xyz="0.2 0 -0.04"/>
-      <geometry>
-        <sphere radius="0.04"/>
-      </geometry>
-      <surface>
-        <friction>
-          <ode>
-            <mu>0</mu>
-            <mu2>0</mu2>
-            <slip1>1.0</slip1>
-            <slip2>1.0</slip2>
-          </ode>
-        </friction>
-      </surface>
-    </collision>
-    <visual name="caster_front_visual">
-      <origin rpy=" 0 0 0" xyz="0.2 0 -0.04"/>
-      <geometry>
-        <sphere radius="0.04"/>
-      </geometry>
-    </visual> -->
     </link>
   <link name = "caster_front">
@@ -112,5 +36,5 @@
       <!-- <origin rpy=" 0 0 0" xyz="0.2 0 -0.04"/> -->
       <geometry>
-        <sphere radius="0.04"/>
+        <sphere radius="0.05"/>
       </geometry>
       <surface>
@@ -128,5 +52,5 @@
       <!-- <origin rpy=" 0 0 0" xyz="0.2 0 -0.04"/> -->
       <geometry>
-        <sphere radius="0.04"/>
+        <sphere radius="0.05"/>
       </geometry>
     </visual>
@@ -171,3 +95,30 @@
     <child link="sensor_laser"/>
   </joint>
+<!-- Camera -->
+  <link name="camera">
+  <collision>
+    <origin xyz="0 0 0" rpy="0 0 0"/>
+    <geometry>
+      <box size="${cameraSize} ${cameraSize} ${cameraSize}"/>
+    </geometry>
+  </collision>
+  <visual>
+    <origin xyz="0 0 0" rpy="0 0 0"/>
+    <geometry>
+      <box size="${cameraSize} ${cameraSize} ${cameraSize}"/>
+    </geometry>
+    <material name="blue"/>
+  </visual>
+  <inertial>
+    <mass value="${cameraMass}" />
+    <origin xyz="0 0 0" rpy="0 0 0"/>
+    <box_inertia m="${cameraMass}" x="${cameraSize}" y="${cameraSize}" z="${cameraSize}" />
+  </inertial>
+</link>
+<joint name="camera_joint" type="fixed">
+  <axis xyz="0.0 1.0 0.0"/>
+  <origin xyz="0.175 0.0 0.127" rpy="0.0 0.0 0.0"/>
+  <parent link="link_chassis"/>
+  <child link="camera"/>
+</joint>
 </robot>
